Commit message: imported changes fabrics-private

File: src/fabrics_sim/models/robots/urdf/kuka_allegro/kuka_allegro_sim.urdf (robot description, URDF)
Before this commit: robot kuka_allegro, 31 links, 30 joints
Links:
- link allegro_mount: geometry 
- link iiwa7_link_0: mass 0.564 -> 0.88556; geometry collision mesh filename=visual/link_base.stl; visual mesh filename=visual/link_base.stl
- link iiwa7_link_1: mass 3.4525 -> 2.382; geometry collision mesh filename=visual/link1.stl; visual mesh filename=visual/link1.stl
- link iiwa7_link_2: mass 3.4821 -> 1.869; geometry collision mesh filename=visual/link2.stl; visual mesh filename=visual/link2.stl
- link iiwa7_link_3: mass 4.05623 -> 1.6383; geometry collision mesh filename=visual/link3.stl; visual mesh filename=visual/link3.stl
- link iiwa7_link_4: mass 3.4822 -> 1.7269; geometry collision mesh filename=visual/link4.stl; visual mesh filename=visual/link4.stl
- link iiwa7_link_5: mass 2.1633 -> 1.3203; geometry collision mesh filename=visual/link5.stl; visual mesh filename=visual/link5.stl
- link iiwa7_link_6: mass 2.3466 -> 1.325; geometry collision mesh filename=visual/link6.stl; visual mesh filename=visual/link6.stl
- link iiwa7_link_7: mass 3.129 -> 0.17; geometry collision mesh filename=collisions/end_tool.stl; visual mesh filename=visual/link7.stl
- link iiwa7_link_ee: mass 1e-7 -> None
- link index_link_0: mass 0.005 -> 0.044; geometry collision mesh filename=visual/mcp_joint.stl; visual mesh filename=visual/mcp_joint.stl
- link index_link_1: mass 0.005 -> 0.032; geometry collision mesh filename=visual/pip.stl; visual mesh filename=visual/pip.stl
- link index_link_2: mass 0.05 -> 0.037; geometry collision mesh filename=visual/dip.stl; visual mesh filename=visual/dip.stl
- link index_link_3: mass 0.11 -> 0.016; geometry collision mesh filename=visual/fingertip.stl; visual mesh filename=visual/fingertip.stl
- link middle_biotac_tip: mass 0.1 -> 0.04
- link middle_link_0: mass 0.1 -> 0.044; geometry collision mesh filename=visual/mcp_joint.stl; visual mesh filename=visual/mcp_joint.stl
- link middle_link_1: mass 0.1 -> 0.032; geometry collision mesh filename=visual/pip.stl; visual mesh filename=visual/pip.stl
- link middle_link_2: mass 0.1 -> 0.037; geometry collision mesh filename=visual/dip.stl; visual mesh filename=visual/dip.stl
- link middle_link_3: mass 0.1 -> 0.016; geometry collision mesh filename=visual/fingertip.stl; visual mesh filename=visual/fingertip.stl
- link palm_link: mass 0.4154 -> 0.237; geometry collision mesh filename=visual/palm_lower.stl; visual mesh filename=visual/palm_lower.stl
- link ring_biotac_tip: mass 0.1 -> 0.04
- link ring_link_0: mass 0.1 -> 0.044; geometry collision mesh filename=visual/mcp_joint.stl; visual mesh filename=visual/mcp_joint.stl
- link ring_link_1: mass 0.1 -> 0.032; geometry collision mesh filename=visual/pip.stl; visual mesh filename=visual/pip.stl
- link ring_link_2: mass 0.1 -> 0.037; geometry collision mesh filename=visual/dip.stl; visual mesh filename=visual/dip.stl
- link ring_link_3: mass 0.1 -> 0.016; geometry collision mesh filename=visual/fingertip.stl; visual mesh filename=visual/fingertip.stl
- link thumb_biotac_tip: mass 0.1 -> 0.04
- link thumb_link_0: mass 0.1 -> 0.032; geometry collision mesh filename=visual/pip.stl; visual mesh filename=visual/pip.stl
- link thumb_link_1: mass 0.1 -> 0.003; geometry collision mesh filename=visual/thumb_pip.stl; visual mesh filename=visual/thumb_pip.stl
- link thumb_link_2: mass 0.1 -> 0.038; geometry collision mesh filename=visual/thumb_dip.stl; visual mesh filename=visual/thumb_dip.stl
- link thumb_link_3: mass 0.1 -> 0.049; geometry collision mesh filename=visual/thumb_fingertip.stl; visual mesh filename=visual/thumb_fingertip.stl
Joints:
- removed joint iiwa7_allegro
- removed joint iiwa7_joint_ee
- added joint iiwa7_to_allegro_fixed: type fixed, parent iiwa7_link_ee, child allegro_mount, origin xyz=0.06 -0.04 0.01 rpy=3.14159 0 0
- added joint joint_eef: type fixed, parent iiwa7_link_7, child iiwa7_link_ee, origin xyz=0 0 0 rpy=0 0 0
- joint allegro_mount_joint: origin xyz=-0.008219 -0.02063 0.08086 rpy=0 -1.5708 0.785398 -> xyz=0 0 0 rpy=0 0 0
- joint iiwa7_joint_1: limit lower=-2.96705972839 upper=2.96705972839 effort=300 velocity=10 -> lower=-6.283185307179586 upper=6.283185307179586 effort=50 velocity=3.14; origin xyz=0 0 0.1575 rpy=0 0 0 -> xyz=0 0 0.267 rpy=0 0 0
- joint iiwa7_joint_2: limit lower=-2.09439510239 upper=2.09439510239 effort=300 velocity=10 -> lower=-2.059 upper=2.0944 effort=50 velocity=3.14; origin xyz=0 0 0.1825 rpy=1.57079632679   0 3.14159265359 -> xyz=0 0 0 rpy=-1.5708 0 0
- joint iiwa7_joint_3: limit lower=-2.96705972839 upper=2.96705972839 effort=300 velocity=10 -> lower=-6.283185307179586 upper=6.283185307179586 effort=30 velocity=3.14; origin xyz=0 0.184 0 rpy=1.57079632679 0 3.14159265359 -> xyz=0 -0.293 0 rpy=1.5708 0 0
- joint iiwa7_joint_4: limit lower=-2.09439510239 upper=2.09439510239 effort=300 velocity=10 -> lower=-0.19198 upper=3.927 effort=30 velocity=3.14; origin xyz=0 0 0.216 rpy=1.57079632679 0 0 -> xyz=0.0525 0 0 rpy=1.5708 0 0
- joint iiwa7_joint_5: limit lower=-2.96705972839 upper=2.96705972839 effort=300 velocity=10 -> lower=-6.283185307179586 upper=6.283185307179586 effort=30 velocity=3.14; origin xyz=0 0.184 0 rpy=-1.57079632679 3.14159265359 0 -> xyz=0.0775 -0.3425 0 rpy=1.5708 0 0
- joint iiwa7_joint_6: limit lower=-2.09439510239 upper=2.09439510239 effort=300 velocity=10 -> lower=-1.69297 upper=3.141592653589793 effort=20 velocity=3.14; origin xyz=0 0.06070 0.216 rpy=1.57079632679 0 0 -> xyz=0 0 0 rpy=1.5708 0 0
- joint iiwa7_joint_7: limit lower=-3.05432619099 upper=3.05432619099 effort=300 velocity=10 -> lower=-6.283185307179586 upper=6.283185307179586 effort=20 velocity=3.14; origin xyz=0 0.081 0.06070 rpy=-1.57079632679 3.14159265359 0 -> xyz=0.076 0.097 0 rpy=-1.5708 0 0
- joint index_biotac_tip_joint: origin xyz=0.055 0.015 0 rpy=0 0 0.436319444444  -> xyz=0 0 0 rpy=0 0 0
- joint index_joint_0: axis 0 0 1 -> 0 0 -1; limit lower=-0.558488888889 upper=0.558488888889 effort=0.35 velocity=6.283 -> lower=-0.314 upper=2.23 effort=0.95 velocity=8.48; origin xyz=0.0514302 -0.03632 -0.0113 rpy=3.1415 -1.57075 -0.0872638888889 -> xyz=-0.0070952496528625457958 0.023057756134899472233 -0.01872240357846021927 rpy=1.5707963267948950037 1.5707963267948945596 0
- joint index_joint_1: axis 0 0 1 -> 0 0 -1; limit lower=-0.279244444444 upper=1.727825 effort=0.35 velocity=6.283 -> lower=-1.047 upper=1.047 effort=0.95 velocity=8.48; origin xyz=0.0 0.0 0.0 rpy=3.1415 -1.57075 1.57075 -> xyz=-0.012200000000000007713 0.038099999999999994982 0.014500000000000000736 rpy=-1.570796326794896558 -1.0065212660796336576e-15 1.5707963267948943376
- joint index_joint_2: axis 0 0 1 -> 0 0 -1; limit lower=-0.279244444444 upper=1.727825 effort=0.35 velocity=6.283 -> lower=-0.506 upper=1.885 effort=0.95 velocity=8.48; origin xyz=0.054 0.0 0.0 rpy=0.0 0.0 0.0 -> xyz=0.01499999999999996822 0.014299999999999904801 -0.012999999999999824196 rpy=1.5707963267948958919 -1.570796326794896336 0
- joint index_joint_3: axis 0 0 1 -> 0 0 -1; limit lower=-0.279244444444 upper=1.727825 effort=0.35 velocity=6.283 -> lower=-0.366 upper=2.042 effort=0.95 velocity=8.48; origin xyz=0.0384 0.0 0.0 rpy=0.0 0.0 0.0 -> xyz=-4.0880582495572692636e-09 -0.036100004210367367397 0.00020000000000007858714 rpy=4.5935029425113685044e-17 -2.8730071914463794583e-16 4.4395481053923607589e-32
- joint middle_biotac_tip_joint: origin xyz=0.055 0.015 0 rpy=0 0 0.436319444444  -> xyz=0 0 0 rpy=0 0 0
- joint middle_joint_0: axis 0 0 1 -> 0 0 -1; limit lower=-0.558488888889 upper=0.558488888889 effort=0.35 velocity=6.283 -> lower=-0.314 upper=2.23 effort=0.95 velocity=8.48; origin xyz=0.0537375 0.0087771 -0.0113 rpy=3.1415 -1.57075 0 -> xyz=-0.0070952496528625388569 -0.022392243865100525113 -0.018722403578460229678 rpy=1.570796326794896558 1.570796326794896558 0
- joint middle_joint_1: axis 0 0 1 -> 0 0 -1; limit lower=-0.279244444444 upper=1.727825 effort=0.35 velocity=6.283 -> lower=-1.047 upper=1.047 effort=0.95 velocity=8.48; origin xyz=0.0 0.0 0.0 rpy=3.1415 -1.57075 1.57075 -> xyz=-0.012200000000000019856 0.038099999999999981104 0.01450000000000000594 rpy=-1.570796326794896558 -1.0065212760057939085e-15 1.5707963267948943376
- joint middle_joint_2: axis 0 0 1 -> 0 0 -1; limit lower=-0.279244444444 upper=1.727825 effort=0.35 velocity=6.283 -> lower=-0.506 upper=1.885 effort=0.95 velocity=8.48; origin xyz=0.054 0.0 0.0 rpy=0.0 0.0 0.0 -> xyz=0.014999999999999975159 0.014300000000000000211 -0.013000000000000018485 rpy=1.5707963267948958919 -1.570796326794896336 0
- joint middle_joint_3: axis 0 0 1 -> 0 0 -1; limit lower=-0.279244444444 upper=1.727825 effort=0.35 velocity=6.283 -> lower=-0.366 upper=2.042 effort=0.95 velocity=8.48; origin xyz=0.0384 0.0 0.0 rpy=0.0 0.0 0.0 -> xyz=1.0061396160665481148e-16 -0.036099999999999854428 0.00020000000000007858714 rpy=4.5935029425113654229e-17 -2.8730071914463794583e-16 1.4408183216511868558e-31
- joint ring_biotac_tip_joint: origin xyz=0.055 0.015 0 rpy=0 0 0.436319444444  -> xyz=0 0 0 rpy=0 0 0
- joint ring_joint_0: axis 0 0 1 -> 0 0 -1; limit lower=-0.558488888889 upper=0.558488888889 effort=0.35 velocity=6.283 -> lower=-0.314 upper=2.23 effort=0.95 velocity=8.48; origin xyz=0.0514302 0.0538749 -0.0113 rpy=3.1415 -1.57075 0.0872638888889 -> xyz=-0.0070952454426398371343 -0.067842243865100515521 -0.018722407666402932774 rpy=1.5707963267948950037 1.5707963267948945596 0
- joint ring_joint_1: axis 0 0 1 -> 0 0 -1; limit lower=-0.279244444444 upper=1.727825 effort=0.35 velocity=6.283 -> lower=-1.047 upper=1.047 effort=0.95 velocity=8.48; origin xyz=0.0 0.0 0.0 rpy=3.1415 -1.57075 1.57075 -> xyz=-0.012200000000000004244 0.038100000000000001921 0.014499999999999999001 rpy=-1.570796326794896558 -1.0065212660796360242e-15 1.5707963267948943376
- joint ring_joint_2: axis 0 0 1 -> 0 0 -1; limit lower=-0.279244444444 upper=1.727825 effort=0.35 velocity=6.283 -> lower=-0.506 upper=1.885 effort=0.95 velocity=8.48; origin xyz=0.054 0.0 0.0 rpy=0.0 0.0 0.0 -> xyz=0.014999999999999971689 0.014299999999999951639 -0.012999999999999959505 rpy=1.5707963267948958919 -1.570796326794896336 0
- joint ring_joint_3: axis 0 0 1 -> 0 0 -1; limit lower=-0.279244444444 upper=1.727825 effort=0.35 velocity=6.283 -> lower=-0.366 upper=2.042 effort=0.95 velocity=8.48; origin xyz=0.0384 0.0 0.0 rpy=0.0 0.0 0.0 -> xyz=9.7144514654701197287e-17 -0.036099999999999868305 0.00020000000000007511769 rpy=4.5935029425113685044e-17 -2.8730071914463799514e-16 1.5565411607615035382e-32
- joint thumb_biotac_tip_joint: origin xyz=0.07 0.01 0 rpy=0 0 0.436319444444  -> xyz=0 0 0 rpy=0 0 0
- joint thumb_joint_0: axis 0 0 1 -> 0 0 -1; limit lower=0.279244444444 upper=1.57075 effort=0.35 velocity=6.283 -> lower=-0.349 upper=2.094 effort=0.95 velocity=8.48; origin xyz=-0.0367482 -0.0081281 -0.0295 rpy=-1.57075 -1.57075 1.48348611111 -> xyz=-0.069395249652862533996 -0.0012422438651005258004 -0.021622403578460215601 rpy=-8.2381766464939424156e-17 1.5707963267948956698 0
- joint thumb_joint_1: axis 0 0 1 -> 0 0 -1; limit lower=-0.331602777778 upper=1.15188333333 effort=0.35 velocity=6.283 -> lower=-0.47 upper=2.443 effort=0.95 velocity=8.48; origin xyz=0.005 0.0 0.0 rpy=1.57075 0 0 -> xyz=-2.7755575615628913511e-17 0.014300000000000005415 -0.013000000000000011546 rpy=1.5707963267948958919 -1.570796326794896336 0
- joint thumb_joint_2: axis 0 0 1 -> 0 0 -1; limit lower=-0.279244444444 upper=1.727825 effort=0.35 velocity=6.283 -> lower=-1.20 upper=1.90 effort=0.95 velocity=8.48; origin xyz=0 0 0.0554 rpy=3.1415 -1.57075 0.0 -> xyz=0 0.014499999999999966041 -0.017000000000000053263 rpy=-1.570796326794896558 1.6050198443300131245e-46 -1.9721522630516624601e-31
- joint thumb_joint_3: axis 0 0 1 -> 0 0 -1; limit lower=-0.279244444444 upper=1.76273055556 effort=0.35 velocity=6.283 -> lower=-1.34 upper=1.88 effort=0.95 velocity=8.48; origin xyz=0.0514 0.0 0.0 rpy=0.0 0.0 0.0 -> xyz=-1.249000902703301108e-16 0.046599999999999863753 0.00019999999999997710581 rpy=1.5063958491491781023e-44 5.4234187233935260503e-31 3.141592653589793116

Commit message: changes urdf and usd for orientation

File: src/fabrics_sim/models/robots/urdf/kuka_allegro/kuka_allegro.urdf (robot description, URDF)
Before this commit: robot kuka_allegro, 52 links, 51 joints
Links:
- link iiwa7_link_ee: mass None -> 0.
Joints:
- removed joint joint_eef
- added joint iiwa7_joint_ee: type fixed, parent iiwa7_link_7, child iiwa7_link_ee, origin xyz=0 0 0 rpy=0 0 0
- joint iiwa7_joint_1: origin xyz=0 0 0.267 rpy=0 0 0 -> xyz=-0.0 -0.0 0.267 rpy=0.0 0.0 3.141592653589793
- joint iiwa7_joint_2: limit lower=-2.967 upper=2.967 effort=50 velocity=3.14 -> lower=-2.059 upper=2.0944 effort=50 velocity=3.14
- joint iiwa7_joint_2_sphere2: origin xyz=0 -0.065 0 rpy=0 0 0 -> xyz=0 0.15 0 rpy=0 0 0
- joint iiwa7_joint_2_sphere3: origin xyz=0 -0.19 0 rpy=0 0 0 -> xyz=0 0.25 0 rpy=0 0 0
- joint iiwa7_joint_4: limit lower=-2.967 upper=2.967 effort=30 velocity=3.14 -> lower=-0.19198 upper=3.927 effort=30 velocity=3.14
- joint iiwa7_joint_4_sphere2: origin xyz=0.04 -0.17 0 rpy=0 0 0 -> xyz=0 0.15 0 rpy=0 0 0
- joint iiwa7_joint_4_sphere3: origin xyz=0.055 -0.26 0 rpy=0 0 0 -> xyz=0 0.25 0 rpy=0 0 0
- joint iiwa7_joint_6: limit lower=-2.094 upper=2.094 effort=20 velocity=3.14 -> lower=-1.69297 upper=3.141592653589793 effort=20 velocity=3.14
- joint iiwa7_joint_6_sphere2: origin xyz=0.065 0.033 0.02 rpy=0 0 0 -> xyz=0 0. 0.05 rpy=0 0 0
- joint index_link_1_joint_sphere2: origin xyz=-0.0061 0.019 0.0073 rpy=0 0 0 -> xyz=0.027 0.0 0. rpy=0 0 0; parent index_link_0 -> index_link_1
- joint index_link_3_joint_sphere2: origin xyz=0 0 0 rpy=0 0 0 -> xyz=0.035 0.005 0. rpy=0 0 0
- joint middle_link_1_joint_sphere2: origin xyz=-0.0061 0.019 0.0073 rpy=0 0 0 -> xyz=0.027 0.0 0. rpy=0 0 0; parent middle_link_0 -> middle_link_1
- joint middle_link_3_joint_sphere2: origin xyz=0 0 0 rpy=0 0 0 -> xyz=0.035 0.005 0. rpy=0 0 0
- joint palm_link_joint_sphere2: origin xyz=-0.0035 0.0115 -0.0094 rpy=0 0 0 -> xyz=0 0.01 -0.05 rpy=0 0 0
- joint ring_link_1_joint_sphere2: origin xyz=-0.0061 0.0191 0.0072 rpy=0 0 0 -> xyz=0.027 0.0 0. rpy=0 0 0; parent ring_link_0 -> ring_link_1
- joint ring_link_3_joint_sphere2: origin xyz=0 0 0 rpy=0 0 0 -> xyz=0.035 0.005 0. rpy=0 0 0
- joint thumb_link_2_joint_sphere2: origin xyz=0 0.0072 -0.0065 rpy=0 0 0 -> xyz=0.025 0.0 0. rpy=0 0 0; parent thumb_link_0 -> thumb_link_2
- joint thumb_link_3_joint_sphere2: origin xyz=0 0.023 0 rpy=0 0 0 -> xyz=0.025 0.0 0. rpy=0 0 0; parent thumb_link_2 -> thumb_link_3
- joint thumb_link_3_joint_sphere3: origin xyz=0 0 0 rpy=0 0 0 -> xyz=0. 0. 0. rpy=0 0 0

File: src/fabrics_sim/models/robots/urdf/kuka_allegro/kuka_allegro_sim.urdf (robot description, URDF)
Before this commit: robot kuka_allegro, 31 links, 30 joints
Links:
- link iiwa7_link_ee: mass None -> 1e-7
Joints:
- removed joint joint_eef
- added joint iiwa7_joint_ee: type fixed, parent iiwa7_link_7, child iiwa7_link_ee, origin xyz=0 0 0 rpy=0 0 0
- joint iiwa7_joint_1: origin xyz=0 0 0.267 rpy=0 0 0 -> xyz=-0.0 -0.0 0.267 rpy=0.0 0.0 3.141592653589793
