Commit message: updated for 41 collisison spheres

File: src/fabrics_sim/models/robots/urdf/kuka_allegro/kuka_allegro.urdf (robot description, URDF)
Before this commit: robot kuka_allegro, 52 links, 51 joints
Links:
- removed link iiwa7_link_2_sphere2
- removed link iiwa7_link_2_sphere3
- removed link iiwa7_link_4_sphere2
- removed link iiwa7_link_4_sphere3
- removed link iiwa7_link_6_sphere2
- removed link index_link_1_sphere2
- removed link index_link_3_sphere2
- removed link middle_link_1_sphere2
- removed link middle_link_3_sphere2
- removed link palm_link_sphere2
- removed link ring_link_1_sphere2
- removed link ring_link_3_sphere2
- removed link thumb_link_2_sphere2
- removed link thumb_link_3_sphere2
- removed link thumb_link_3_sphere3
- added link iiwa7_link_0_sphere_0; collision sphere radius=0.106865; visual sphere radius=0.106865
- added link iiwa7_link_1_sphere_0; collision sphere radius=0.106078; visual sphere radius=0.106078
- added link iiwa7_link_2_sphere_0; collision sphere radius=0.102232; visual sphere radius=0.102232
- added link iiwa7_link_2_sphere_1; collision sphere radius=0.085125; visual sphere radius=0.085125
- added link iiwa7_link_3_sphere_0; collision sphere radius=0.10456; visual sphere radius=0.10456
- added link iiwa7_link_4_sphere_0; collision sphere radius=0.093645; visual sphere radius=0.093645
- added link iiwa7_link_4_sphere_1; collision sphere radius=0.073883; visual sphere radius=0.073883
- added link iiwa7_link_5_sphere_0; collision sphere radius=0.074265; visual sphere radius=0.074265
- added link iiwa7_link_5_sphere_1; collision sphere radius=0.075691; visual sphere radius=0.075691
- added link iiwa7_link_6_sphere_0; collision sphere radius=0.093184; visual sphere radius=0.093184
- added link iiwa7_link_7_sphere_0; collision sphere radius=0.046394; visual sphere radius=0.046394
- added link index_link_0_sphere_0; collision sphere radius=0.030195; visual sphere radius=0.030195
- added link index_link_0_sphere_1; collision sphere radius=0.029524; visual sphere radius=0.029524
- added link index_link_1_sphere_0; collision sphere radius=0.025406; visual sphere radius=0.025406
- added link index_link_2_sphere_0; collision sphere radius=0.025943; visual sphere radius=0.025943
- added link index_link_2_sphere_1; collision sphere radius=0.025238; visual sphere radius=0.025238
- added link index_link_3_sphere_0; collision sphere radius=0.025322; visual sphere radius=0.025322
- added link index_link_3_sphere_1; collision sphere radius=0.023613; visual sphere radius=0.023613
- added link middle_link_0_sphere_0; collision sphere radius=0.030195; visual sphere radius=0.030195
- added link middle_link_0_sphere_1; collision sphere radius=0.029524; visual sphere radius=0.029524
- added link middle_link_1_sphere_0; collision sphere radius=0.025406; visual sphere radius=0.025406
- added link middle_link_2_sphere_0; collision sphere radius=0.025943; visual sphere radius=0.025943
- added link middle_link_2_sphere_1; collision sphere radius=0.025238; visual sphere radius=0.025238
- added link middle_link_3_sphere_0; collision sphere radius=0.025322; visual sphere radius=0.025322
- added link middle_link_3_sphere_1; collision sphere radius=0.023613; visual sphere radius=0.023613
- added link palm_link_sphere_0; collision sphere radius=0.064833; visual sphere radius=0.064833
- added link palm_link_sphere_1; collision sphere radius=0.063931; visual sphere radius=0.063931
- added link ring_link_0_sphere_0; collision sphere radius=0.030195; visual sphere radius=0.030195
- added link ring_link_0_sphere_1; collision sphere radius=0.029524; visual sphere radius=0.029524
- added link ring_link_1_sphere_0; collision sphere radius=0.025406; visual sphere radius=0.025406
- added link ring_link_2_sphere_0; collision sphere radius=0.025943; visual sphere radius=0.025943
- added link ring_link_2_sphere_1; collision sphere radius=0.025238; visual sphere radius=0.025238
- added link ring_link_3_sphere_0; collision sphere radius=0.025322; visual sphere radius=0.025322
- added link ring_link_3_sphere_1; collision sphere radius=0.023613; visual sphere radius=0.023613
- added link thumb_link_0_sphere_0; collision sphere radius=0.025406; visual sphere radius=0.025406
- added link thumb_link_1_sphere_0; collision sphere radius=0.017487; visual sphere radius=0.017487
- added link thumb_link_1_sphere_1; collision sphere radius=0.017227; visual sphere radius=0.017227
- added link thumb_link_2_sphere_0; collision sphere radius=0.027454; visual sphere radius=0.027454
- added link thumb_link_2_sphere_1; collision sphere radius=0.025244; visual sphere radius=0.025244
- added link thumb_link_3_sphere_0; collision sphere radius=0.024778; visual sphere radius=0.024778
- added link thumb_link_3_sphere_1; collision sphere radius=0.027507; visual sphere radius=0.027507
- link iiwa7_link_0: geometry visual mesh filename=visual/link_base.stl
- link iiwa7_link_1: geometry visual mesh filename=visual/link1.stl
- link iiwa7_link_2: geometry visual mesh filename=visual/link2.stl
- link iiwa7_link_3: geometry visual mesh filename=visual/link3.stl
- link iiwa7_link_4: geometry visual mesh filename=visual/link4.stl
- link iiwa7_link_5: geometry visual mesh filename=visual/link5.stl
- link iiwa7_link_6: geometry visual mesh filename=visual/link6.stl
- link iiwa7_link_7: geometry visual mesh filename=visual/link7.stl
- link iiwa7_link_ee: mass 0. -> 1e-7
- link index_link_0: geometry visual mesh filename=visual/mcp_joint.stl
- link index_link_1: geometry visual mesh filename=visual/pip.stl
- link index_link_2: geometry visual mesh filename=visual/dip.stl
- link index_link_3: geometry visual mesh filename=visual/fingertip.stl
- link middle_link_0: geometry visual mesh filename=visual/mcp_joint.stl
- link middle_link_1: geometry visual mesh filename=visual/pip.stl
- link middle_link_2: geometry visual mesh filename=visual/dip.stl
- link middle_link_3: geometry visual mesh filename=visual/fingertip.stl
- link palm_link: geometry visual mesh filename=visual/palm_lower.stl
- link ring_link_0: geometry visual mesh filename=visual/mcp_joint.stl
- link ring_link_1: geometry visual mesh filename=visual/pip.stl
- link ring_link_2: geometry visual mesh filename=visual/dip.stl
- link ring_link_3: geometry visual mesh filename=visual/fingertip.stl
- link thumb_link_0: geometry visual mesh filename=visual/pip.stl
- link thumb_link_1: geometry visual mesh filename=visual/thumb_pip.stl
- link thumb_link_2: geometry visual mesh filename=visual/thumb_dip.stl
- link thumb_link_3: geometry visual mesh filename=visual/thumb_fingertip.stl
Joints:
- removed joint iiwa7_joint_2_sphere2
- removed joint iiwa7_joint_2_sphere3
- removed joint iiwa7_joint_4_sphere2
- removed joint iiwa7_joint_4_sphere3
- removed joint iiwa7_joint_6_sphere2
- removed joint index_link_1_joint_sphere2
- removed joint index_link_3_joint_sphere2
- removed joint middle_link_1_joint_sphere2
- removed joint middle_link_3_joint_sphere2
- removed joint palm_link_joint_sphere2
- removed joint ring_link_1_joint_sphere2
- removed joint ring_link_3_joint_sphere2
- removed joint thumb_link_2_joint_sphere2
- removed joint thumb_link_3_joint_sphere2
- removed joint thumb_link_3_joint_sphere3
- added joint iiwa7_link_0_sphere_0_joint: type fixed, parent iiwa7_link_0, child iiwa7_link_0_sphere_0, origin xyz=0.0011192172081857226 -0.00021905044747053354 0.06825173159942649 rpy=0 0 0
- added joint iiwa7_link_1_sphere_0_joint: type fixed, parent iiwa7_link_1, child iiwa7_link_1_sphere_0, origin xyz=-6.100736480189614e-05 0.005716614252139976 -0.02496277297813876 rpy=0 0 0
- added joint iiwa7_link_2_sphere_0_joint: type fixed, parent iiwa7_link_2, child iiwa7_link_2_sphere_0, origin xyz=0.0003252776992805183 -0.13172392472836197 0.03221276276974082 rpy=0 0 0
- added joint iiwa7_link_2_sphere_1_joint: type fixed, parent iiwa7_link_2, child iiwa7_link_2_sphere_1, origin xyz=0.00046227769928051834 -0.028333924728361957 0.08911076276974081 rpy=0 0 0
- added joint iiwa7_link_3_sphere_0_joint: type fixed, parent iiwa7_link_3, child iiwa7_link_3_sphere_0, origin xyz=0.03083603806713227 -0.00960750634898807 -0.03273608703856688 rpy=0 0 0
- added joint iiwa7_link_4_sphere_0_joint: type fixed, parent iiwa7_link_4, child iiwa7_link_4_sphere_0, origin xyz=0.07776186234366894 -0.09730177018964291 0.017834635922193528 rpy=0 0 0
- added joint iiwa7_link_4_sphere_1_joint: type fixed, parent iiwa7_link_4, child iiwa7_link_4_sphere_1, origin xyz=0.02324486234366894 -0.01871277018964291 0.08140563592219352 rpy=0 0 0
- added joint iiwa7_link_5_sphere_0_joint: type fixed, parent iiwa7_link_5, child iiwa7_link_5_sphere_0, origin xyz=0.00043856173980236056 0.01788517520344257 -0.1294335997161865 rpy=0 0 0
- added joint iiwa7_link_5_sphere_1_joint: type fixed, parent iiwa7_link_5, child iiwa7_link_5_sphere_1, origin xyz=-0.00035343826019763945 0.054711175203442576 -0.019401599716186525 rpy=0 0 0
- added joint iiwa7_link_6_sphere_0_joint: type fixed, parent iiwa7_link_6, child iiwa7_link_6_sphere_0, origin xyz=0.04119180196136403 0.019968113325854582 0.013544495331668054 rpy=0 0 0
- added joint iiwa7_link_7_sphere_0_joint: type fixed, parent iiwa7_link_7, child iiwa7_link_7_sphere_0, origin xyz=0.00010096233355998993 -0.006664624187827111 -0.013500000350177288 rpy=0 0 0
- added joint index_link_0_sphere_0_joint: type fixed, parent index_link_0, child index_link_0_sphere_0, origin xyz=-0.02709780039471551 0.0389927757203814 0.01822488284482244 rpy=0 0 0
- added joint index_link_0_sphere_1_joint: type fixed, parent index_link_0, child index_link_0_sphere_1, origin xyz=-0.004758800394715509 0.012566775720381403 0.013422882844822438 rpy=0 0 0
- added joint index_link_1_sphere_0_joint: type fixed, parent index_link_1, child index_link_1_sphere_0, origin xyz=0.007550909541881593 -4.070128988430469e-05 -0.011544538941221595 rpy=0 0 0
- added joint index_link_2_sphere_0_joint: type fixed, parent index_link_2, child index_link_2_sphere_0, origin xyz=-0.000160444468868157 -0.0064222726501808585 0.011588584740962232 rpy=0 0 0
- added joint index_link_2_sphere_1_joint: type fixed, parent index_link_2, child index_link_2_sphere_1, origin xyz=0.007172555531131843 -0.032630272650180855 0.01444458474096223 rpy=0 0 0
- added joint index_link_3_sphere_0_joint: type fixed, parent index_link_3, child index_link_3_sphere_0, origin xyz=4.163860108443026e-05 -0.006146559023194272 0.017471736681818326 rpy=0 0 0
- added joint index_link_3_sphere_1_joint: type fixed, parent index_link_3, child index_link_3_sphere_1, origin xyz=-0.0011503613989155698 -0.029922559023194274 0.015378736681818325 rpy=0 0 0
- added joint middle_link_0_sphere_0_joint: type fixed, parent middle_link_0, child middle_link_0_sphere_0, origin xyz=-0.02709780039471551 0.0389927757203814 0.018224882844822442 rpy=0 0 0
- added joint middle_link_0_sphere_1_joint: type fixed, parent middle_link_0, child middle_link_0_sphere_1, origin xyz=-0.004758800394715509 0.012566775720381403 0.013422882844822443 rpy=0 0 0
- added joint middle_link_1_sphere_0_joint: type fixed, parent middle_link_1, child middle_link_1_sphere_0, origin xyz=0.007550909541881593 -4.070128988429948e-05 -0.011544538941221595 rpy=0 0 0
- added joint middle_link_2_sphere_0_joint: type fixed, parent middle_link_2, child middle_link_2_sphere_0, origin xyz=-0.000160444468868157 -0.006422272650180845 0.011588584740962228 rpy=0 0 0
- added joint middle_link_2_sphere_1_joint: type fixed, parent middle_link_2, child middle_link_2_sphere_1, origin xyz=0.007172555531131843 -0.03263027265018084 0.014444584740962227 rpy=0 0 0
- added joint middle_link_3_sphere_0_joint: type fixed, parent middle_link_3, child middle_link_3_sphere_0, origin xyz=4.163860108442332e-05 -0.006146559023194286 0.017471736681818322 rpy=0 0 0
- added joint middle_link_3_sphere_1_joint: type fixed, parent middle_link_3, child middle_link_3_sphere_1, origin xyz=-0.0011503613989155767 -0.029922559023194288 0.015378736681818323 rpy=0 0 0
- added joint palm_link_sphere_0_joint: type fixed, parent palm_link, child palm_link_sphere_0, origin xyz=-0.04827191059877636 -0.06074232003230608 -0.010488238606124346 rpy=0 0 0
- added joint palm_link_sphere_1_joint: type fixed, parent palm_link, child palm_link_sphere_1, origin xyz=-0.05024191059877636 -0.007173320032306078 -0.011593238606124346 rpy=0 0 0
- added joint ring_link_0_sphere_0_joint: type fixed, parent ring_link_0, child ring_link_0_sphere_0, origin xyz=-0.0270978003947155 0.0389927757203814 0.018224882844822442 rpy=0 0 0
- added joint ring_link_0_sphere_1_joint: type fixed, parent ring_link_0, child ring_link_0_sphere_1, origin xyz=-0.004758800394715502 0.012566775720381403 0.013422882844822443 rpy=0 0 0
- added joint ring_link_1_sphere_0_joint: type fixed, parent ring_link_1, child ring_link_1_sphere_0, origin xyz=0.007550909541881597 -4.070128988431336e-05 -0.011544538941221595 rpy=0 0 0
- added joint ring_link_2_sphere_0_joint: type fixed, parent ring_link_2, child ring_link_2_sphere_0, origin xyz=-0.00016044446886815354 -0.006422272650180845 0.011588584740962228 rpy=0 0 0
- added joint ring_link_2_sphere_1_joint: type fixed, parent ring_link_2, child ring_link_2_sphere_1, origin xyz=0.007172555531131847 -0.03263027265018084 0.014444584740962227 rpy=0 0 0
- added joint ring_link_3_sphere_0_joint: type fixed, parent ring_link_3, child ring_link_3_sphere_0, origin xyz=4.1638601084428525e-05 -0.006146559023194272 0.017471736681818326 rpy=0 0 0
- added joint ring_link_3_sphere_1_joint: type fixed, parent ring_link_3, child ring_link_3_sphere_1, origin xyz=-0.0011503613989155715 -0.029922559023194274 0.015378736681818325 rpy=0 0 0
- added joint thumb_link_0_sphere_0_joint: type fixed, parent thumb_link_0, child thumb_link_0_sphere_0, origin xyz=-0.007449090458118406 -4.070128988429428e-05 -0.011544538941221594 rpy=0 0 0
- added joint thumb_link_1_sphere_0_joint: type fixed, parent thumb_link_1, child thumb_link_1_sphere_0, origin xyz=0.0012950003509032925 0.011532999999999469 -0.008354259973414538 rpy=0 0 0
- added joint thumb_link_1_sphere_1_joint: type fixed, parent thumb_link_1, child thumb_link_1_sphere_1, origin xyz=-0.0014139996490967074 -0.011603000000000531 -0.008646259973414536 rpy=0 0 0
- added joint thumb_link_2_sphere_0_joint: type fixed, parent thumb_link_2, child thumb_link_2_sphere_0, origin xyz=-0.0019106185261045356 0.011429891791562823 -0.013659642629872498 rpy=0 0 0
- added joint thumb_link_2_sphere_1_joint: type fixed, parent thumb_link_2, child thumb_link_2_sphere_1, origin xyz=-0.00015661852610453567 0.040609891791562824 -0.0163776426298725 rpy=0 0 0
- added joint thumb_link_3_sphere_0_joint: type fixed, parent thumb_link_3, child thumb_link_3_sphere_0, origin xyz=0.0028524943401055784 -0.008154384363043058 -0.01422490549846478 rpy=0 0 0
- added joint thumb_link_3_sphere_1_joint: type fixed, parent thumb_link_3, child thumb_link_3_sphere_1, origin xyz=0.0006064943401055782 -0.038899384363043056 -0.013859905498464779 rpy=0 0 0

Commit message: Hand vertical mount

File: src/fabrics_sim/models/robots/urdf/kuka_allegro/kuka_allegro.urdf (robot description, URDF)
Before this commit: robot kuka_allegro, 78 links, 77 joints
Links:
- link iiwa7_link_0_sphere_0: geometry visual sphere radius=0.106865
- link iiwa7_link_1_sphere_0: geometry visual sphere radius=0.106078
- link iiwa7_link_2_sphere_0: geometry visual sphere radius=0.102232
- link iiwa7_link_2_sphere_1: geometry visual sphere radius=0.085125
- link iiwa7_link_3_sphere_0: geometry visual sphere radius=0.10456
- link iiwa7_link_4_sphere_0: geometry visual sphere radius=0.093645
- link iiwa7_link_4_sphere_1: geometry visual sphere radius=0.073883
- link iiwa7_link_5_sphere_0: geometry visual sphere radius=0.074265
- link iiwa7_link_5_sphere_1: geometry visual sphere radius=0.075691
- link iiwa7_link_6_sphere_0: geometry visual sphere radius=0.074547
- link iiwa7_link_7_sphere_0: geometry visual sphere radius=0.037115
- link index_link_0_sphere_0: geometry visual sphere radius=0.018117
- link index_link_0_sphere_1: geometry visual sphere radius=0.0177144
- link index_link_1_sphere_0: geometry visual sphere radius=0.0152436
- link index_link_2_sphere_0: geometry visual sphere radius=0.0155658
- link index_link_2_sphere_1: geometry visual sphere radius=0.0151428
- link index_link_3_sphere_0: geometry visual sphere radius=0.0151932
- link index_link_3_sphere_1: geometry visual sphere radius=0.0141678
- link middle_link_0_sphere_0: geometry visual sphere radius=0.018117
- link middle_link_0_sphere_1: geometry visual sphere radius=0.0177144
- link middle_link_1_sphere_0: geometry visual sphere radius=0.0152436
- link middle_link_2_sphere_0: geometry visual sphere radius=0.0155658
- link middle_link_2_sphere_1: geometry visual sphere radius=0.0151428
- link middle_link_3_sphere_0: geometry visual sphere radius=0.0151932
- link middle_link_3_sphere_1: geometry visual sphere radius=0.0141678
- link palm_link_sphere_0: geometry visual sphere radius=0.0388998
- link palm_link_sphere_1: geometry visual sphere radius=0.0383586
- link ring_link_0_sphere_0: geometry visual sphere radius=0.018117
- link ring_link_0_sphere_1: geometry visual sphere radius=0.0177144
- link ring_link_1_sphere_0: geometry visual sphere radius=0.0152436
- link ring_link_2_sphere_0: geometry visual sphere radius=0.0155658
- link ring_link_2_sphere_1: geometry visual sphere radius=0.0151428
- link ring_link_3_sphere_0: geometry visual sphere radius=0.0151932
- link ring_link_3_sphere_1: geometry visual sphere radius=0.0141678
- link thumb_link_0_sphere_0: geometry visual sphere radius=0.0152436
- link thumb_link_1_sphere_0: geometry visual sphere radius=0.0104922
- link thumb_link_1_sphere_1: geometry visual sphere radius=0.0103362
- link thumb_link_2_sphere_0: geometry visual sphere radius=0.0164724
- link thumb_link_2_sphere_1: geometry visual sphere radius=0.0151464
- link thumb_link_3_sphere_0: geometry visual sphere radius=0.0148668
- link thumb_link_3_sphere_1: geometry visual sphere radius=0.0165042
Joints:
- joint allegro_mount_joint: origin xyz=0 0 0 rpy=0 0 0 -> xyz=-0.07 -0.065 -0.09 rpy=0 1.57 3.14
- joint index_biotac_tip_joint: origin xyz=0 0 0 rpy=0 0 0 -> xyz=-0.01 -0.04 0.016 rpy=3.14 0 -1.54
- joint middle_biotac_tip_joint: origin xyz=0 0 0 rpy=0 0 0 -> xyz=-0.01 -0.04 0.016 rpy=3.14 0 -1.54
- joint palm_x_joint: origin xyz=0.25 0. 0. rpy=0. 0. 0. -> xyz=0.25 0. 0. rpy=3.14 0. 0.
- joint palm_x_neg_joint: origin xyz=-0.25 0. 0. rpy=0. 0. 0. -> xyz=-0.25 0. 0. rpy=3.14 0. 0.
- joint palm_y_joint: origin xyz=0. 0.25 0. rpy=0. 0. 0. -> xyz=0. -0.25 0. rpy=3.14 0. 0.
- joint palm_y_neg_joint: origin xyz=0. -0.25 0. rpy=0. 0. 0. -> xyz=0. 0.25 0. rpy=3.14 0. 0.
- joint palm_z_joint: origin xyz=0. 0. 0.25 rpy=0. 0. 0. -> xyz=0. 0. -0.25 rpy=3.14 0. 0.
- joint palm_z_neg_joint: origin xyz=0. 0. -0.25 rpy=0. 0. 0. -> xyz=0. 0. 0.25 rpy=3.14 0. 0.
- joint ring_biotac_tip_joint: origin xyz=0 0 0 rpy=0 0 0 -> xyz=-0.01 -0.04 0.016 rpy=3.14 0 -1.54
- joint thumb_biotac_tip_joint: origin xyz=0 0 0 rpy=0 0 0 -> xyz=-0.01 -0.05 -0.0125 rpy=3.14 0 -1.54

File: src/fabrics_sim/models/robots/urdf/kuka_allegro/kuka_allegro_sim.urdf (robot description, URDF)
Before this commit: robot kuka_allegro, 31 links, 30 joints
Joints:
- joint allegro_mount_joint: origin xyz=0 0 0 rpy=0 0 0 -> xyz=-0.07 -0.065 -0.09 rpy=0 1.57 3.14
- joint index_biotac_tip_joint: origin xyz=0 0 0 rpy=0 0 0 -> xyz=-0.01 -0.04 0.016 rpy=3.14 0 -1.54
- joint middle_biotac_tip_joint: origin xyz=0 0 0 rpy=0 0 0 -> xyz=-0.01 -0.04 0.016 rpy=3.14 0 -1.54
- joint ring_biotac_tip_joint: origin xyz=0 0 0 rpy=0 0 0 -> xyz=-0.01 -0.04 0.016 rpy=3.14 0 -1.54
- joint thumb_biotac_tip_joint: origin xyz=0 0 0 rpy=0 0 0 -> xyz=-0.01 -0.05 -0.0125 rpy=3.14 0 -1.54
