Commit message: kuka_leaphand  changes

File: src/fabrics_sim/models/robots/urdf/kuka_allegro/kuka_allegro.urdf (robot description, URDF)
Before this commit: robot kuka_allegro, 78 links, 77 joints
Links:
- removed link iiwa7_link_0_sphere_0
- removed link iiwa7_link_1_sphere_0
- removed link iiwa7_link_2_sphere_0
- removed link iiwa7_link_2_sphere_1
- removed link iiwa7_link_3_sphere_0
- removed link iiwa7_link_4_sphere_0
- removed link iiwa7_link_4_sphere_1
- removed link iiwa7_link_5_sphere_0
- removed link iiwa7_link_5_sphere_1
- removed link iiwa7_link_6_sphere_0
- removed link iiwa7_link_7_sphere_0
- added link _virtual_palm_link, mass 0.04
- added link iiwa7_link_2_sphere2
- added link iiwa7_link_2_sphere3
- added link iiwa7_link_4_sphere2
- added link iiwa7_link_4_sphere3
- added link iiwa7_link_6_sphere2
- link allegro_mount: geometry collision mesh filename=meshes/allegro_mount.stl; visual mesh filename=meshes/allegro_mount.stl
- link iiwa7_link_0: mass 0.88556 -> 0.564; geometry collision mesh filename=meshes/link_0.stl; visual mesh filename=meshes/link_0.stl
- link iiwa7_link_1: mass 2.382 -> 3.4525; geometry collision mesh filename=meshes/link_1.stl; visual mesh filename=meshes/link_1.stl
- link iiwa7_link_2: mass 1.869 -> 3.4821; geometry collision mesh filename=meshes/link_2.stl; visual mesh filename=meshes/link_2.stl
- link iiwa7_link_3: mass 1.6383 -> 4.05623; geometry collision mesh filename=meshes/link_3.stl; visual mesh filename=meshes/link_3.stl
- link iiwa7_link_4: mass 1.7269 -> 3.4822; geometry collision mesh filename=meshes/link_4.stl; visual mesh filename=meshes/link_4.stl
- link iiwa7_link_5: mass 1.3203 -> 2.1633; geometry collision mesh filename=meshes/link_5.stl; visual mesh filename=meshes/link_5.stl
- link iiwa7_link_6: mass 1.325 -> 2.3466; geometry collision mesh filename=meshes/link_6.stl; visual mesh filename=meshes/link_6.stl
- link iiwa7_link_7: mass 0.17 -> 3.129; geometry collision mesh filename=meshes/link_7.stl; visual mesh filename=meshes/link_7.stl
- link index_link_0: geometry collision mesh filename=visual/mcp_joint.stl; visual mesh filename=visual/mcp_joint.stl
- link index_link_1: geometry collision mesh filename=visual/pip.stl; visual mesh filename=visual/pip.stl
- link index_link_2: geometry collision mesh filename=visual/dip.stl; visual mesh filename=visual/dip.stl
- link index_link_3: geometry collision mesh filename=visual/fingertip.stl; visual mesh filename=visual/fingertip.stl
- link middle_link_0: geometry collision mesh filename=visual/mcp_joint.stl; visual mesh filename=visual/mcp_joint.stl
- link middle_link_1: geometry collision mesh filename=visual/pip.stl; visual mesh filename=visual/pip.stl
- link middle_link_2: geometry collision mesh filename=visual/dip.stl; visual mesh filename=visual/dip.stl
- link middle_link_3: geometry collision mesh filename=visual/fingertip.stl; visual mesh filename=visual/fingertip.stl
- link palm_link: geometry collision mesh filename=visual/palm_lower.stl; visual mesh filename=visual/palm_lower.stl
- link ring_link_0: geometry collision mesh filename=visual/mcp_joint.stl; visual mesh filename=visual/mcp_joint.stl
- link ring_link_1: geometry collision mesh filename=visual/pip.stl; visual mesh filename=visual/pip.stl
- link ring_link_2: geometry collision mesh filename=visual/dip.stl; visual mesh filename=visual/dip.stl
- link ring_link_3: geometry collision mesh filename=visual/fingertip.stl; visual mesh filename=visual/fingertip.stl
- link thumb_link_0: geometry collision mesh filename=visual/pip.stl; visual mesh filename=visual/pip.stl
- link thumb_link_1: geometry collision mesh filename=visual/thumb_pip.stl; visual mesh filename=visual/thumb_pip.stl
- link thumb_link_2: geometry collision mesh filename=visual/thumb_dip.stl; visual mesh filename=visual/thumb_dip.stl
- link thumb_link_3: geometry collision mesh filename=visual/thumb_fingertip.stl; visual mesh filename=visual/thumb_fingertip.stl
Joints:
- removed joint iiwa7_link_0_sphere_0_joint
- removed joint iiwa7_link_1_sphere_0_joint
- removed joint iiwa7_link_2_sphere_0_joint
- removed joint iiwa7_link_2_sphere_1_joint
- removed joint iiwa7_link_3_sphere_0_joint
- removed joint iiwa7_link_4_sphere_0_joint
- removed joint iiwa7_link_4_sphere_1_joint
- removed joint iiwa7_link_5_sphere_0_joint
- removed joint iiwa7_link_5_sphere_1_joint
- removed joint iiwa7_link_6_sphere_0_joint
- removed joint iiwa7_link_7_sphere_0_joint
- removed joint iiwa7_to_allegro_fixed
- added joint iiwa7_allegro: type fixed, parent iiwa7_link_ee, child allegro_mount, origin xyz=0 0 0 rpy=0 0 0
- added joint iiwa7_joint_2_sphere2: type fixed, parent iiwa7_link_2, child iiwa7_link_2_sphere2, origin xyz=0 0.15 0 rpy=0 0 0, axis 0 0 1
- added joint iiwa7_joint_2_sphere3: type fixed, parent iiwa7_link_2, child iiwa7_link_2_sphere3, origin xyz=0 0.25 0 rpy=0 0 0, axis 0 0 1
- added joint iiwa7_joint_4_sphere2: type fixed, parent iiwa7_link_4, child iiwa7_link_4_sphere2, origin xyz=0 0.15 0 rpy=0 0 0, axis 0 0 1
- added joint iiwa7_joint_4_sphere3: type fixed, parent iiwa7_link_4, child iiwa7_link_4_sphere3, origin xyz=0 0.25 0 rpy=0 0 0, axis 0 0 1
- added joint iiwa7_joint_6_sphere2: type fixed, parent iiwa7_link_6, child iiwa7_link_6_sphere2, origin xyz=0 0. 0.05 rpy=0 0 0, axis 0 0 1
- added joint palm_virtual_joint: type fixed, parent palm_link, child _virtual_palm_link, origin xyz=-0.0425 -0.0375 -0.035 rpy=3.14 0. 0.
- joint allegro_mount_joint: origin xyz=-0.07 -0.065 -0.09 rpy=0 1.57 3.14 -> xyz=0.03 -0.01 0.125 rpy=0 -1.5708 3.925398
- joint iiwa7_joint_1: limit lower=-6.283185307179586 upper=6.283185307179586 effort=50 velocity=3.14 -> lower=-2.96705972839 upper=2.96705972839 effort=300 velocity=10; origin xyz=-0.0 -0.0 0.267 rpy=0.0 0.0 3.141592653589793 -> xyz=0 0 0.1575 rpy=0 0 0
- joint iiwa7_joint_2: limit lower=-2.059 upper=2.0944 effort=50 velocity=3.14 -> lower=-2.09439510239 upper=2.09439510239 effort=300 velocity=10; origin xyz=0 0 0 rpy=-1.5708 0 0 -> xyz=0 0 0.1825 rpy=1.57079632679   0 3.14159265359
- joint iiwa7_joint_3: limit lower=-6.283185307179586 upper=6.283185307179586 effort=30 velocity=3.14 -> lower=-2.96705972839 upper=2.96705972839 effort=300 velocity=10; origin xyz=0 -0.293 0 rpy=1.5708 0 0 -> xyz=0 0.184 0 rpy=1.57079632679 0 3.14159265359
- joint iiwa7_joint_4: limit lower=-0.19198 upper=3.927 effort=30 velocity=3.14 -> lower=-2.09439510239 upper=2.09439510239 effort=300 velocity=10; origin xyz=0.0525 0 0 rpy=1.5708 0 0 -> xyz=0 0 0.216 rpy=1.57079632679 0 0
- joint iiwa7_joint_5: limit lower=-6.283185307179586 upper=6.283185307179586 effort=30 velocity=3.14 -> lower=-2.96705972839 upper=2.96705972839 effort=300 velocity=10; origin xyz=0.0775 -0.3425 0 rpy=1.5708 0 0 -> xyz=0 0.184 0 rpy=-1.57079632679 3.14159265359 0
- joint iiwa7_joint_6: limit lower=-1.69297 upper=3.141592653589793 effort=20 velocity=3.14 -> lower=-2.09439510239 upper=2.09439510239 effort=300 velocity=10; origin xyz=0 0 0 rpy=1.5708 0 0 -> xyz=0 0.06070 0.216 rpy=1.57079632679 0 0
- joint iiwa7_joint_7: limit lower=-6.283185307179586 upper=6.283185307179586 effort=20 velocity=3.14 -> lower=-3.05432619099 upper=3.05432619099 effort=300 velocity=10; origin xyz=0.076 0.097 0 rpy=-1.5708 0 0 -> xyz=0 0.081 0.06070 rpy=-1.57079632679 3.14159265359 0
- joint iiwa7_joint_ee: origin xyz=0 0 0 rpy=0 0 0 -> xyz=0 0 0.071 rpy=0 0 0
- joint palm_x_joint: parent palm_link -> _virtual_palm_link
- joint palm_x_neg_joint: parent palm_link -> _virtual_palm_link
- joint palm_y_joint: origin xyz=0. -0.25 0. rpy=3.14 0. 0. -> xyz=0. 0.25 0. rpy=3.14 0. 0.; parent palm_link -> _virtual_palm_link
- joint palm_y_neg_joint: origin xyz=0. 0.25 0. rpy=3.14 0. 0. -> xyz=0. -0.25 0. rpy=3.14 0. 0.; parent palm_link -> _virtual_palm_link
- joint palm_z_joint: origin xyz=0. 0. -0.25 rpy=3.14 0. 0. -> xyz=0. 0. 0.25 rpy=3.14 0. 0.; parent palm_link -> _virtual_palm_link
- joint palm_z_neg_joint: origin xyz=0. 0. 0.25 rpy=3.14 0. 0. -> xyz=0. 0. -0.25 rpy=3.14 0. 0.; parent palm_link -> _virtual_palm_link

File: src/fabrics_sim/models/robots/urdf/kuka_allegro/kuka_allegro_sim.urdf (robot description, URDF)
Before this commit: robot kuka_allegro, 31 links, 30 joints
Links:
- link allegro_mount: geometry collision mesh filename=meshes/allegro_mount.stl; visual mesh filename=meshes/allegro_mount.stl
- link iiwa7_link_0: mass 0.88556 -> 0.564; geometry collision mesh filename=meshes/link_0.stl; visual mesh filename=meshes/link_0.stl
- link iiwa7_link_1: mass 2.382 -> 3.4525; geometry collision mesh filename=meshes/link_1.stl; visual mesh filename=meshes/link_1.stl
- link iiwa7_link_2: mass 1.869 -> 3.4821; geometry collision mesh filename=meshes/link_2.stl; visual mesh filename=meshes/link_2.stl
- link iiwa7_link_3: mass 1.6383 -> 4.05623; geometry collision mesh filename=meshes/link_3.stl; visual mesh filename=meshes/link_3.stl
- link iiwa7_link_4: mass 1.7269 -> 3.4822; geometry collision mesh filename=meshes/link_4.stl; visual mesh filename=meshes/link_4.stl
- link iiwa7_link_5: mass 1.3203 -> 2.1633; geometry collision mesh filename=meshes/link_5.stl; visual mesh filename=meshes/link_5.stl
- link iiwa7_link_6: mass 1.325 -> 2.3466; geometry collision mesh filename=meshes/link_6.stl; visual mesh filename=meshes/link_6.stl
- link iiwa7_link_7: mass 0.17 -> 3.129; geometry collision mesh filename=meshes/link_7.stl; visual mesh filename=meshes/link_7.stl
Joints:
- removed joint iiwa7_to_allegro_fixed
- added joint iiwa7_allegro: type fixed, parent iiwa7_link_ee, child allegro_mount, origin xyz=0 0 0 rpy=0 0 0
- joint allegro_mount_joint: origin xyz=-0.07 -0.065 -0.09 rpy=0 1.57 3.14 -> xyz=0.03 -0.01 0.125 rpy=0 -1.5708 3.925398
- joint iiwa7_joint_1: limit lower=-6.283185307179586 upper=6.283185307179586 effort=50 velocity=3.14 -> lower=-2.96705972839 upper=2.96705972839 effort=300 velocity=10; origin xyz=-0.0 -0.0 0.267 rpy=0.0 0.0 3.141592653589793 -> xyz=0 0 0.1575 rpy=0 0 0
- joint iiwa7_joint_2: limit lower=-2.059 upper=2.0944 effort=50 velocity=3.14 -> lower=-2.09439510239 upper=2.09439510239 effort=300 velocity=10; origin xyz=0 0 0 rpy=-1.5708 0 0 -> xyz=0 0 0.1825 rpy=1.57079632679   0 3.14159265359
- joint iiwa7_joint_3: limit lower=-6.283185307179586 upper=6.283185307179586 effort=30 velocity=3.14 -> lower=-2.96705972839 upper=2.96705972839 effort=300 velocity=10; origin xyz=0 -0.293 0 rpy=1.5708 0 0 -> xyz=0 0.184 0 rpy=1.57079632679 0 3.14159265359
- joint iiwa7_joint_4: limit lower=-0.19198 upper=3.927 effort=30 velocity=3.14 -> lower=-2.09439510239 upper=2.09439510239 effort=300 velocity=10; origin xyz=0.0525 0 0 rpy=1.5708 0 0 -> xyz=0 0 0.216 rpy=1.57079632679 0 0
- joint iiwa7_joint_5: limit lower=-6.283185307179586 upper=6.283185307179586 effort=30 velocity=3.14 -> lower=-2.96705972839 upper=2.96705972839 effort=300 velocity=10; origin xyz=0.0775 -0.3425 0 rpy=1.5708 0 0 -> xyz=0 0.184 0 rpy=-1.57079632679 3.14159265359 0
- joint iiwa7_joint_6: limit lower=-1.69297 upper=3.141592653589793 effort=20 velocity=3.14 -> lower=-2.09439510239 upper=2.09439510239 effort=300 velocity=10; origin xyz=0 0 0 rpy=1.5708 0 0 -> xyz=0 0.06070 0.216 rpy=1.57079632679 0 0
- joint iiwa7_joint_7: limit lower=-6.283185307179586 upper=6.283185307179586 effort=20 velocity=3.14 -> lower=-3.05432619099 upper=3.05432619099 effort=300 velocity=10; origin xyz=0.076 0.097 0 rpy=-1.5708 0 0 -> xyz=0 0.081 0.06070 rpy=-1.57079632679 3.14159265359 0
- joint iiwa7_joint_ee: origin xyz=0 0 0 rpy=0 0 0 -> xyz=0 0 0.071 rpy=0 0 0

Commit message: smaller and lower woorkspace

File: src/fabrics_sim/models/robots/urdf/kuka_allegro/kuka_allegro.urdf (robot description, URDF)
Before this commit: robot kuka_allegro, 73 links, 72 joints
Links:
- removed link iiwa7_link_2_sphere2
- removed link iiwa7_link_2_sphere3
- removed link iiwa7_link_4_sphere2
- removed link iiwa7_link_4_sphere3
- removed link iiwa7_link_6_sphere2
- added link iiwa7_link_0_sphere_0; visual sphere radius=0.106865
- added link iiwa7_link_1_sphere_0; visual sphere radius=0.106078
- added link iiwa7_link_2_sphere_0; visual sphere radius=0.102232
- added link iiwa7_link_2_sphere_1; visual sphere radius=0.085125
- added link iiwa7_link_3_sphere_0; visual sphere radius=0.10456
- added link iiwa7_link_4_sphere_0; visual sphere radius=0.093645
- added link iiwa7_link_4_sphere_1; visual sphere radius=0.073883
- added link iiwa7_link_5_sphere_0; visual sphere radius=0.074265
- added link iiwa7_link_5_sphere_1; visual sphere radius=0.075691
- added link iiwa7_link_6_sphere_0; visual sphere radius=0.074547
- added link iiwa7_link_7_sphere_0; visual sphere radius=0.037115
- link allegro_mount: geometry 
- link iiwa7_link_0: mass 0.564 -> 0.88556; geometry collision mesh filename=visual/link_base.stl; visual mesh filename=visual/link_base.stl
- link iiwa7_link_1: mass 3.4525 -> 2.382; geometry collision mesh filename=visual/link1.stl; visual mesh filename=visual/link1.stl
- link iiwa7_link_2: mass 3.4821 -> 1.869; geometry collision mesh filename=visual/link2.stl; visual mesh filename=visual/link2.stl
- link iiwa7_link_3: mass 4.05623 -> 1.6383; geometry collision mesh filename=visual/link3.stl; visual mesh filename=visual/link3.stl
- link iiwa7_link_4: mass 3.4822 -> 1.7269; geometry collision mesh filename=visual/link4.stl; visual mesh filename=visual/link4.stl
- link iiwa7_link_5: mass 2.1633 -> 1.3203; geometry collision mesh filename=visual/link5.stl; visual mesh filename=visual/link5.stl
- link iiwa7_link_6: mass 2.3466 -> 1.325; geometry collision mesh filename=visual/link6.stl; visual mesh filename=visual/link6.stl
- link iiwa7_link_7: mass 3.129 -> 0.17; geometry collision mesh filename=visual/link7.stl; visual mesh filename=visual/link7.stl
Joints:
- removed joint iiwa7_allegro
- removed joint iiwa7_joint_2_sphere2
- removed joint iiwa7_joint_2_sphere3
- removed joint iiwa7_joint_4_sphere2
- removed joint iiwa7_joint_4_sphere3
- removed joint iiwa7_joint_6_sphere2
- added joint iiwa7_link_0_sphere_0_joint: type fixed, parent iiwa7_link_0, child iiwa7_link_0_sphere_0, origin xyz=0.0011192172081857226 -0.00021905044747053354 0.06825173159942649 rpy=0 0 0
- added joint iiwa7_link_1_sphere_0_joint: type fixed, parent iiwa7_link_1, child iiwa7_link_1_sphere_0, origin xyz=-6.100736480189614e-05 0.005716614252139976 -0.02496277297813876 rpy=0 0 0
- added joint iiwa7_link_2_sphere_0_joint: type fixed, parent iiwa7_link_2, child iiwa7_link_2_sphere_0, origin xyz=0.0003252776992805183 -0.13172392472836197 0.03221276276974082 rpy=0 0 0
- added joint iiwa7_link_2_sphere_1_joint: type fixed, parent iiwa7_link_2, child iiwa7_link_2_sphere_1, origin xyz=0.00046227769928051834 -0.028333924728361957 0.08911076276974081 rpy=0 0 0
- added joint iiwa7_link_3_sphere_0_joint: type fixed, parent iiwa7_link_3, child iiwa7_link_3_sphere_0, origin xyz=0.03083603806713227 -0.00960750634898807 -0.03273608703856688 rpy=0 0 0
- added joint iiwa7_link_4_sphere_0_joint: type fixed, parent iiwa7_link_4, child iiwa7_link_4_sphere_0, origin xyz=0.07776186234366894 -0.09730177018964291 0.017834635922193528 rpy=0 0 0
- added joint iiwa7_link_4_sphere_1_joint: type fixed, parent iiwa7_link_4, child iiwa7_link_4_sphere_1, origin xyz=0.02324486234366894 -0.01871277018964291 0.08140563592219352 rpy=0 0 0
- added joint iiwa7_link_5_sphere_0_joint: type fixed, parent iiwa7_link_5, child iiwa7_link_5_sphere_0, origin xyz=0.00043856173980236056 0.01788517520344257 -0.1294335997161865 rpy=0 0 0
- added joint iiwa7_link_5_sphere_1_joint: type fixed, parent iiwa7_link_5, child iiwa7_link_5_sphere_1, origin xyz=-0.00035343826019763945 0.054711175203442576 -0.019401599716186525 rpy=0 0 0
- added joint iiwa7_link_6_sphere_0_joint: type fixed, parent iiwa7_link_6, child iiwa7_link_6_sphere_0, origin xyz=0.04119180196136403 0.019968113325854582 0.013544495331668054 rpy=0 0 0
- added joint iiwa7_link_7_sphere_0_joint: type fixed, parent iiwa7_link_7, child iiwa7_link_7_sphere_0, origin xyz=0.00010096233355998993 -0.006664624187827111 -0.013500000350177288 rpy=0 0 0
- added joint iiwa7_to_allegro_fixed: type fixed, parent iiwa7_link_ee, child allegro_mount, origin xyz=0.06 -0.04 0.01 rpy=3.14159 0 0
- joint allegro_mount_joint: origin xyz=0.03 -0.01 0.125 rpy=0 -1.5708 3.925398 -> xyz=0 0 0 rpy=0 0 0
- joint iiwa7_joint_1: limit lower=-2.96705972839 upper=2.96705972839 effort=300 velocity=10 -> lower=-6.283185307179586 upper=6.283185307179586 effort=50 velocity=3.14; origin xyz=0 0 0.1575 rpy=0 0 0 -> xyz=-0.0 -0.0 0.267 rpy=0.0 0.0 3.141592653589793
- joint iiwa7_joint_2: limit lower=-2.09439510239 upper=2.09439510239 effort=300 velocity=10 -> lower=-2.059 upper=2.0944 effort=50 velocity=3.14; origin xyz=0 0 0.1825 rpy=1.57079632679   0 3.14159265359 -> xyz=0 0 0 rpy=-1.5708 0 0
- joint iiwa7_joint_3: limit lower=-2.96705972839 upper=2.96705972839 effort=300 velocity=10 -> lower=-6.283185307179586 upper=6.283185307179586 effort=30 velocity=3.14; origin xyz=0 0.184 0 rpy=1.57079632679 0 3.14159265359 -> xyz=0 -0.293 0 rpy=1.5708 0 0
- joint iiwa7_joint_4: limit lower=-2.09439510239 upper=2.09439510239 effort=300 velocity=10 -> lower=-0.19198 upper=3.927 effort=30 velocity=3.14; origin xyz=0 0 0.216 rpy=1.57079632679 0 0 -> xyz=0.0525 0 0 rpy=1.5708 0 0
- joint iiwa7_joint_5: limit lower=-2.96705972839 upper=2.96705972839 effort=300 velocity=10 -> lower=-6.283185307179586 upper=6.283185307179586 effort=30 velocity=3.14; origin xyz=0 0.184 0 rpy=-1.57079632679 3.14159265359 0 -> xyz=0.0775 -0.3425 0 rpy=1.5708 0 0
- joint iiwa7_joint_6: limit lower=-2.09439510239 upper=2.09439510239 effort=300 velocity=10 -> lower=-1.69297 upper=3.141592653589793 effort=20 velocity=3.14; origin xyz=0 0.06070 0.216 rpy=1.57079632679 0 0 -> xyz=0 0 0 rpy=1.5708 0 0
- joint iiwa7_joint_7: limit lower=-3.05432619099 upper=3.05432619099 effort=300 velocity=10 -> lower=-6.283185307179586 upper=6.283185307179586 effort=20 velocity=3.14; origin xyz=0 0.081 0.06070 rpy=-1.57079632679 3.14159265359 0 -> xyz=0.076 0.097 0 rpy=-1.5708 0 0
- joint iiwa7_joint_ee: origin xyz=0 0 0.071 rpy=0 0 0 -> xyz=0 0 0 rpy=0 0 0

File: src/fabrics_sim/models/robots/urdf/kuka_allegro/kuka_allegro_sim.urdf (robot description, URDF)
Before this commit: robot kuka_allegro, 31 links, 30 joints
Links:
- link allegro_mount: geometry 
- link iiwa7_link_0: mass 0.564 -> 0.88556; geometry collision mesh filename=visual/link_base.stl; visual mesh filename=visual/link_base.stl
- link iiwa7_link_1: mass 3.4525 -> 2.382; geometry collision mesh filename=visual/link1.stl; visual mesh filename=visual/link1.stl
- link iiwa7_link_2: mass 3.4821 -> 1.869; geometry collision mesh filename=visual/link2.stl; visual mesh filename=visual/link2.stl
- link iiwa7_link_3: mass 4.05623 -> 1.6383; geometry collision mesh filename=visual/link3.stl; visual mesh filename=visual/link3.stl
- link iiwa7_link_4: mass 3.4822 -> 1.7269; geometry collision mesh filename=visual/link4.stl; visual mesh filename=visual/link4.stl
- link iiwa7_link_5: mass 2.1633 -> 1.3203; geometry collision mesh filename=visual/link5.stl; visual mesh filename=visual/link5.stl
- link iiwa7_link_6: mass 2.3466 -> 1.325; geometry collision mesh filename=visual/link6.stl; visual mesh filename=visual/link6.stl
- link iiwa7_link_7: mass 3.129 -> 0.17; geometry collision mesh filename=visual/link7.stl; visual mesh filename=visual/link7.stl
Joints:
- removed joint iiwa7_allegro
- added joint iiwa7_to_allegro_fixed: type fixed, parent iiwa7_link_ee, child allegro_mount, origin xyz=0.06 -0.04 0.01 rpy=3.14159 0 0
- joint allegro_mount_joint: origin xyz=0.03 -0.01 0.125 rpy=0 -1.5708 3.925398 -> xyz=0 0 0 rpy=0 0 0
- joint iiwa7_joint_1: limit lower=-2.96705972839 upper=2.96705972839 effort=300 velocity=10 -> lower=-6.283185307179586 upper=6.283185307179586 effort=50 velocity=3.14; origin xyz=0 0 0.1575 rpy=0 0 0 -> xyz=-0.0 -0.0 0.267 rpy=0.0 0.0 3.141592653589793
- joint iiwa7_joint_2: limit lower=-2.09439510239 upper=2.09439510239 effort=300 velocity=10 -> lower=-2.059 upper=2.0944 effort=50 velocity=3.14; origin xyz=0 0 0.1825 rpy=1.57079632679   0 3.14159265359 -> xyz=0 0 0 rpy=-1.5708 0 0
- joint iiwa7_joint_3: limit lower=-2.96705972839 upper=2.96705972839 effort=300 velocity=10 -> lower=-6.283185307179586 upper=6.283185307179586 effort=30 velocity=3.14; origin xyz=0 0.184 0 rpy=1.57079632679 0 3.14159265359 -> xyz=0 -0.293 0 rpy=1.5708 0 0
- joint iiwa7_joint_4: limit lower=-2.09439510239 upper=2.09439510239 effort=300 velocity=10 -> lower=-0.19198 upper=3.927 effort=30 velocity=3.14; origin xyz=0 0 0.216 rpy=1.57079632679 0 0 -> xyz=0.0525 0 0 rpy=1.5708 0 0
- joint iiwa7_joint_5: limit lower=-2.96705972839 upper=2.96705972839 effort=300 velocity=10 -> lower=-6.283185307179586 upper=6.283185307179586 effort=30 velocity=3.14; origin xyz=0 0.184 0 rpy=-1.57079632679 3.14159265359 0 -> xyz=0.0775 -0.3425 0 rpy=1.5708 0 0
- joint iiwa7_joint_6: limit lower=-2.09439510239 upper=2.09439510239 effort=300 velocity=10 -> lower=-1.69297 upper=3.141592653589793 effort=20 velocity=3.14; origin xyz=0 0.06070 0.216 rpy=1.57079632679 0 0 -> xyz=0 0 0 rpy=1.5708 0 0
- joint iiwa7_joint_7: limit lower=-3.05432619099 upper=3.05432619099 effort=300 velocity=10 -> lower=-6.283185307179586 upper=6.283185307179586 effort=20 velocity=3.14; origin xyz=0 0.081 0.06070 rpy=-1.57079632679 3.14159265359 0 -> xyz=0.076 0.097 0 rpy=-1.5708 0 0
- joint iiwa7_joint_ee: origin xyz=0 0 0.071 rpy=0 0 0 -> xyz=0 0 0 rpy=0 0 0

Commit message: acc and vel lims

File: src/fabrics_sim/models/robots/urdf/kuka_allegro/kuka_allegro.urdf (robot description, URDF)
Before this commit: robot kuka_allegro, 79 links, 78 joints
Links:
- link index_link_3_sphere_1: geometry visual sphere radius=0.0161678
- link middle_link_3_sphere_1: geometry visual sphere radius=0.0161678
- link ring_link_3_sphere_1: geometry visual sphere radius=0.0161678
Joints:
- joint index_link_3_sphere_1_joint: origin xyz=-0.0011503613989155698 -0.029922559023194274 0.015378736681818325 rpy=0 0 0 -> xyz=-0.0011503613989155698 -0.034922559023194274 0.015378736681818325 rpy=0 0 0
- joint middle_link_3_sphere_1_joint: origin xyz=-0.0011503613989155767 -0.029922559023194288 0.015378736681818323 rpy=0 0 0 -> xyz=-0.0011503613989155767 -0.034922559023194274 0.015378736681818323 rpy=0 0 0
- joint ring_link_3_sphere_1_joint: origin xyz=-0.0011503613989155715 -0.029922559023194274 0.015378736681818325 rpy=0 0 0 -> xyz=-0.0011503613989155715 -0.034922559023194274 0.015378736681818325 rpy=0 0 0
- joint thumb_link_3_sphere_1_joint: origin xyz=0.0006064943401055782 -0.038899384363043056 -0.013859905498464779 rpy=0 0 0 -> xyz=0.0006064943401055782 -0.04899384363043056 -0.013859905498464779 rpy=0 0 0
